File: keyboard.kicad_pcb (KiCad board)
At the start: 2 copper layers, 263.5 x 82.5 mm, 93 parts, among them U1 ProMicro

Commit message: hotswap ver
Parts:
- removed D_~{1}: D, Diode_SMD:D_SOD-123
- removed G*** (x2): LOGO, silkscreens:quir_border
- removed K_~{1}: KEYSW, MX_Alps_Hybrid:MXOnly-1U-NoLED
- added D_~1: D, Diode_SMD:D_SOD-123, B.Cu at (253.0, 96.9)
- added K_~1: KEYSW, MX_Hotswap:MX-Hotswap-1U, F.Cu at (244.3, 95.4)
- K_125, K_126, K_127: footprint MX_Alps_Hybrid:MXOnly-1.25U-NoLED -> MX_Hotswap:MX-Hotswap-1.25U
- K_150, K_151, K_152: footprint MX_Alps_Hybrid:MXOnly-1.5U-NoLED -> MX_Hotswap:MX-Hotswap-1.5U
- K_175, K_176: footprint MX_Alps_Hybrid:MXOnly-1.75U-NoLED -> MX_Hotswap:MX-Hotswap-1.75U
- K_2: footprint MX_Alps_Hybrid:MXOnly-2U-NoLED -> MX_Hotswap:MX-Hotswap-2U
- K_225: footprint MX_Alps_Hybrid:MXOnly-2.25U-NoLED -> MX_Hotswap:MX-Hotswap-2.25U
- K_A1, K_B1, K_C1, K_COMMA1, K_D1, K_DOT1, K_E1, K_F1, K_FREE1, K_G1, K_H1, K_I1, K_J1, K_K1, K_L1, K_M1, K_N1, K_O1, K_P1, K_PLUS1, K_Q1, K_R1, K_S1, K_SEMIC1, K_SLASH1, K_SPACE1, K_T1, K_TAB1, K_U1, K_V1, K_W1, K_X1, K_Y1, K_Z1: footprint MX_Alps_Hybrid:MXOnly-1U-NoLED -> MX_Hotswap:MX-Hotswap-1U
- moved D_TAB1 17.5 mm to (80.0, 43.0), turned to 90 degrees
- moved D_Q1 9.72 mm to (82.4, 43.0)
- moved D_125 1.68 mm to (60.9, 58.9)
- moved D_151 1.68 mm to (60.9, 77.9)
Connections:
- U1 pad 1: Net-(U1-Pad1) -> unconnected-(U1-TX0/PD3-Pad1)
- U1 pad 2: Net-(U1-Pad2) -> unconnected-(U1-RX1/PD2-Pad2)
- U1 pad 21: Net-(U1-Pad21) -> unconnected-(U1-VCC-Pad21)
- U1 pad 22: Net-(U1-Pad22) -> unconnected-(U1-RST-Pad22)
- U1 pad 24: Net-(U1-Pad24) -> unconnected-(U1-RAW-Pad24)
Routing:
- net row3: track 263.4 -> 292.7 mm, vias 1 -> 0
- net row1: track 211.7 -> 233.7 mm, vias 1 -> 11
- net Net-(D_TAB1-A): track 44.8 -> 26.0 mm, vias 1 -> 0
- net row2: track 231.1 -> 249.5 mm, vias 1 -> 11
- net Net-(D_~{1-Pad2}): track 8.24 -> 0.00 mm
- net Net-(D_126-A): track 14.9 -> 23.0 mm, vias 0 -> 2
- net Net-(D_150-A): track 15.7 -> 23.2 mm, vias 0 -> 2
- net row0: track 214.9 -> 221.3 mm, vias 0 -> 12
- net Net-(D_~1-A): track 0.00 -> 6.15 mm
- net col11: track 252.2 -> 246.5 mm
- net Net-(D_151-A): track 13.0 -> 8.05 mm
- net Net-(D_175-A): track 17.3 -> 22.2 mm
- net Net-(D_125-A): track 10.7 -> 6.50 mm
- net col3: track 77.2 -> 73.1 mm, vias 0 -> 1
- net Net-(D_2-A): track 15.4 -> 12.1 mm
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
Commit message: updated bom
Parts:
- D_125, D_126, D_127, D_150, D_151, D_152, D_175, D_176, D_2, D_225, D_A1, D_B1, D_C1, D_COMMA1, D_D1, D_DOT1, D_E1, D_F1, D_FREE1, D_G1, D_H1, D_I1, D_J1, D_K1, D_L1, D_M1, D_N1, D_O1, D_P1, D_PLUS1, D_Q1, D_R1, D_S1, D_SEMIC1, D_SLASH1, D_SPACE1, D_T1, D_TAB1, D_U1, D_V1, D_W1, D_X1, D_Y1, D_Z1, D_~1: value D -> 1N4148W
