File: keyboard.kicad_sch (KiCad schematic)
At the start: 91 parts, among them U1 ProMicro

Commit message: hotswap ver
Parts:
- K_125, K_126, K_127: footprint MX_Alps_Hybrid:MXOnly-1.25U-NoLED -> MX_Hotswap:MX-Hotswap-1.25U
- K_150, K_151, K_152: footprint MX_Alps_Hybrid:MXOnly-1.5U-NoLED -> MX_Hotswap:MX-Hotswap-1.5U
- K_175, K_176: footprint MX_Alps_Hybrid:MXOnly-1.75U-NoLED -> MX_Hotswap:MX-Hotswap-1.75U
- K_2: footprint MX_Alps_Hybrid:MXOnly-2U-NoLED -> MX_Hotswap:MX-Hotswap-2U
- K_225: footprint MX_Alps_Hybrid:MXOnly-2.25U-NoLED -> MX_Hotswap:MX-Hotswap-2.25U
- K_A1, K_B1, K_C1, K_COMMA1, K_D1, K_DOT1, K_E1, K_F1, K_FREE1, K_G1, K_H1, K_I1, K_J1, K_K1, K_L1, K_M1, K_N1, K_O1, K_P1, K_PLUS1, K_Q1, K_R1, K_S1, K_SEMIC1, K_SLASH1, K_SPACE1, K_T1, K_TAB1, K_U1, K_V1, K_W1, K_X1, K_Y1, K_Z1, K_~1: footprint MX_Alps_Hybrid:MXOnly-1U-NoLED -> MX_Hotswap:MX-Hotswap-1U

Commit message: updated bom
Parts:
- D_125, D_126, D_127, D_150, D_151, D_152, D_175, D_176, D_2, D_225, D_A1, D_B1, D_C1, D_COMMA1, D_D1, D_DOT1, D_E1, D_F1, D_FREE1, D_G1, D_H1, D_I1, D_J1, D_K1, D_L1, D_M1, D_N1, D_O1, D_P1, D_PLUS1, D_Q1, D_R1, D_S1, D_SEMIC1, D_SLASH1, D_SPACE1, D_T1, D_TAB1, D_U1, D_V1, D_W1, D_X1, D_Y1, D_Z1, D_~1: value D -> 1N4148W; LCSC (none) -> C81598
